File: riliwifi-master/riliwifi-master/riliwifi-master/Hardware/relewifi-2025-05-13_163020/relewifi.kicad_pcb (KiCad board)
At the start: 2 copper layers, 45 parts, among them J10 Screw_Terminal_01x03, J11 Screw_Terminal_01x03, J3 Screw_Terminal_01x03, J4 Screw_Terminal_01x03, J5 Screw_Terminal_01x02, J6 Screw_Terminal_01x03, J7 Screw_Terminal_01x03, J8 Screw_Terminal_01x03, J9 Screw_Terminal_01x03, K1 FINDER-40.52, K2 FINDER-40.52, K3 FINDER-40.52, K4 FINDER-40.52, Q1 Q_NPN_BCE, Q2 Q_NPN_BCE, Q3 Q_NPN_BCE, Q4 Q_NPN_BCE, U1 EL817, U2 EL817, U3 EL817, U4 EL817, U5 L7805, U6 ESP32DevKitv1

Commit message: Para imprimir
Parts:
- removed Q1, Q2, Q4: Q_NPN_BCE, Package_TO_SOT_SMD:SOT-23
- removed the Q3 at (69.9, 58.1)
- added C1: 0,1uF, Capacitor_THT:C_Axial_L3.8mm_D2.6mm_P7.50mm_Horizontal, F.Cu at (261.4, 155.0)
- added C1: 0,1uF, Capacitor_THT:C_Axial_L3.8mm_D2.6mm_P7.50mm_Horizontal, F.Cu at (261.3, 47.7)
- added C2: 0,33uF, Capacitor_THT:C_Axial_L3.8mm_D2.6mm_P7.50mm_Horizontal, F.Cu at (247.0, 155.0)
- added C2: 0,33uF, Capacitor_THT:C_Axial_L3.8mm_D2.6mm_P7.50mm_Horizontal, F.Cu at (246.9, 47.7)
- added D1: D, Diode_SMD:D_SMA, F.Cu at (286.4, 157.5)
- added D1: D, Diode_SMD:D_SMA, F.Cu at (286.3, 50.1)
- added D2: LED, LED_THT:LED_D5.0mm_Clear, F.Cu at (269.3, 157.4)
- added D2: LED, LED_THT:LED_D5.0mm_Clear, F.Cu at (269.2, 50.1)
- added D3: D, Diode_SMD:D_SMA, F.Cu at (285.9, 200.1)
- added D3: D, Diode_SMD:D_SMA, F.Cu at (285.9, 92.8)
- added D4: LED, LED_THT:LED_D5.0mm_Clear, F.Cu at (268.3, 208.1)
- added D4: LED, LED_THT:LED_D5.0mm_Clear, F.Cu at (268.3, 100.8)
- added D5: D, Diode_SMD:D_SMA, F.Cu at (284.2, 66.5)
- added D5: D, Diode_SMD:D_SMA, F.Cu at (284.3, 173.9)
- added D6: LED, LED_THT:LED_D5.0mm_Clear, F.Cu at (267.8, 69.2)
- added D6: LED, LED_THT:LED_D5.0mm_Clear, F.Cu at (267.8, 176.5)
- added D7: D, Diode_SMD:D_SMA, F.Cu at (285.6, 113.0)
- added D7: D, Diode_SMD:D_SMA, F.Cu at (285.7, 220.3)
- added D8: LED, LED_THT:LED_D5.0mm_Clear, F.Cu at (268.3, 227.2)
- added D8: LED, LED_THT:LED_D5.0mm_Clear, F.Cu at (268.2, 119.9)
- added J10: Screw_Terminal_01x03, TerminalBlock:TerminalBlock_Xinya_XY308-2.54-3P_1x03_P2.54mm_Horizontal, F.Cu at (324.8, 172.0)
- added J10: Screw_Terminal_01x03, TerminalBlock:TerminalBlock_Xinya_XY308-2.54-3P_1x03_P2.54mm_Horizontal, F.Cu at (324.7, 64.7)
- added J11: Screw_Terminal_01x03, TerminalBlock:TerminalBlock_Xinya_XY308-2.54-3P_1x03_P2.54mm_Horizontal, F.Cu at (324.8, 181.7)
- added J11: Screw_Terminal_01x03, TerminalBlock:TerminalBlock_Xinya_XY308-2.54-3P_1x03_P2.54mm_Horizontal, F.Cu at (324.7, 74.4)
- added J3: Screw_Terminal_01x03, TerminalBlock:TerminalBlock_Xinya_XY308-2.54-3P_1x03_P2.54mm_Horizontal, F.Cu at (324.8, 45.9)
- added J3: Screw_Terminal_01x03, TerminalBlock:TerminalBlock_Xinya_XY308-2.54-3P_1x03_P2.54mm_Horizontal, F.Cu at (324.8, 153.2)
- added J4: Screw_Terminal_01x03, TerminalBlock:TerminalBlock_Xinya_XY308-2.54-3P_1x03_P2.54mm_Horizontal, F.Cu at (324.7, 220.8)
- added J4: Screw_Terminal_01x03, TerminalBlock:TerminalBlock_Xinya_XY308-2.54-3P_1x03_P2.54mm_Horizontal, F.Cu at (324.7, 113.5)
- added J5: Screw_Terminal_01x02, TerminalBlock:TerminalBlock_bornier-2_P5.08mm, F.Cu at (238.2, 41.2)
- added J5: Screw_Terminal_01x02, TerminalBlock:TerminalBlock_bornier-2_P5.08mm, F.Cu at (238.2, 148.5)
- added J6: Screw_Terminal_01x03, TerminalBlock:TerminalBlock_Xinya_XY308-2.54-3P_1x03_P2.54mm_Horizontal, F.Cu at (324.8, 199.8)
- added J6: Screw_Terminal_01x03, TerminalBlock:TerminalBlock_Xinya_XY308-2.54-3P_1x03_P2.54mm_Horizontal, F.Cu at (324.8, 92.5)
- added J7: Screw_Terminal_01x03, TerminalBlock:TerminalBlock_Xinya_XY308-2.54-3P_1x03_P2.54mm_Horizontal, F.Cu at (324.7, 230.8)
- added J7: Screw_Terminal_01x03, TerminalBlock:TerminalBlock_Xinya_XY308-2.54-3P_1x03_P2.54mm_Horizontal, F.Cu at (324.6, 123.5)
- added J8: Screw_Terminal_01x03, TerminalBlock:TerminalBlock_Xinya_XY308-2.54-3P_1x03_P2.54mm_Horizontal, F.Cu at (324.8, 208.5)
- added J8: Screw_Terminal_01x03, TerminalBlock:TerminalBlock_Xinya_XY308-2.54-3P_1x03_P2.54mm_Horizontal, F.Cu at (324.7, 101.1)
- added J9: Screw_Terminal_01x03, TerminalBlock:TerminalBlock_Xinya_XY308-2.54-3P_1x03_P2.54mm_Horizontal, F.Cu at (324.9, 162.5)
- added J9: Screw_Terminal_01x03, TerminalBlock:TerminalBlock_Xinya_XY308-2.54-3P_1x03_P2.54mm_Horizontal, F.Cu at (324.8, 55.2)
- added K1: FINDER-40.52, Relay_THT:Relay_DPDT_Finder_40.52, F.Cu at (291.6, 43.4)
- added K1: FINDER-40.52, Relay_THT:Relay_DPDT_Finder_40.52, F.Cu at (291.6, 150.7)
- added K2: FINDER-40.52, Relay_THT:Relay_DPDT_Finder_40.52, F.Cu at (291.8, 169.4)
- added K2: FINDER-40.52, Relay_THT:Relay_DPDT_Finder_40.52, F.Cu at (291.8, 62.1)
- added K3: FINDER-40.52, Relay_THT:Relay_DPDT_Finder_40.52, F.Cu at (291.7, 90.4)
- added K3: FINDER-40.52, Relay_THT:Relay_DPDT_Finder_40.52, F.Cu at (291.7, 197.7)
- added K4: FINDER-40.52, Relay_THT:Relay_DPDT_Finder_40.52, F.Cu at (293.3, 111.0)
- added K4: FINDER-40.52, Relay_THT:Relay_DPDT_Finder_40.52, F.Cu at (293.4, 218.3)
- added Q3: MMBT2222A, Package_TO_SOT_SMD:SOT-23, F.Cu at (278.7, 180.4)
- added Q3: MMBT2222A, Package_TO_SOT_SMD:SOT-23, F.Cu at (278.7, 73.1)
- added Q3: MMBT2222A, Package_TO_SOT_SMD:SOT-23, F.Cu at (134.2, 72.6)
- added Q5: MMBT2222A, Package_TO_SOT_SMD:SOT-23, F.Cu at (278.6, 122.7)
- added Q5: MMBT2222A, Package_TO_SOT_SMD:SOT-23, F.Cu at (134.1, 122.3)
- added Q5: MMBT2222A, Package_TO_SOT_SMD:SOT-23, F.Cu at (278.6, 230.1)
- added Q6: MMBT2222A, Package_TO_SOT_SMD:SOT-23, F.Cu at (133.2, 103.4)
- added Q6: MMBT2222A, Package_TO_SOT_SMD:SOT-23, F.Cu at (277.7, 211.2)
- added Q6: MMBT2222A, Package_TO_SOT_SMD:SOT-23, F.Cu at (277.6, 103.9)
- added Q7: MMBT2222A, Package_TO_SOT_SMD:SOT-23, F.Cu at (277.7, 157.0)
- added Q7: MMBT2222A, Package_TO_SOT_SMD:SOT-23, F.Cu at (133.3, 49.2)
- added Q7: MMBT2222A, Package_TO_SOT_SMD:SOT-23, F.Cu at (277.7, 49.7)
- added R1: R, Resistor_SMD:R_0805_2012Metric, F.Cu at (268.4, 94.2)
- added R1: R, Resistor_SMD:R_0805_2012Metric, F.Cu at (268.4, 201.5)
- added R10: R, Resistor_SMD:R_0805_2012Metric, F.Cu at (273.8, 159.1)
- added R10: R, Resistor_SMD:R_0805_2012Metric, F.Cu at (273.8, 51.8)
- added R11: R, Resistor_SMD:R_0805_2012Metric, F.Cu at (273.4, 70.8)
- added R11: R, Resistor_SMD:R_0805_2012Metric, F.Cu at (273.5, 178.1)
- added R12: R, Resistor_SMD:R_0805_2012Metric, F.Cu at (274.5, 230.1)
- added R12: R, Resistor_SMD:R_0805_2012Metric, F.Cu at (274.5, 122.8)
- added R2: R, Resistor_SMD:R_0805_2012Metric, F.Cu at (279.5, 207.7)
- added R2: R, Resistor_SMD:R_0805_2012Metric, F.Cu at (279.5, 100.4)
- added R3: R, Resistor_SMD:R_0805_2012Metric, F.Cu at (270.3, 114.4)
- added R3: R, Resistor_SMD:R_0805_2012Metric, F.Cu at (270.4, 221.7)
- added R4: R, Resistor_SMD:R_0805_2012Metric, F.Cu at (279.3, 176.0)
- added R4: R, Resistor_SMD:R_0805_2012Metric, F.Cu at (279.3, 68.6)
- added R5: R, Resistor_SMD:R_0805_2012Metric, F.Cu at (266.5, 63.8)
- added R5: R, Resistor_SMD:R_0805_2012Metric, F.Cu at (266.5, 171.1)
- added R6: R, Resistor_SMD:R_0805_2012Metric, F.Cu at (270.9, 151.6)
- added R6: R, Resistor_SMD:R_0805_2012Metric, F.Cu at (270.8, 44.3)
- added R7: R, Resistor_SMD:R_0805_2012Metric, F.Cu at (281.9, 158.4)
- added R7: R, Resistor_SMD:R_0805_2012Metric, F.Cu at (281.9, 51.1)
- added R8: R, Resistor_SMD:R_0805_2012Metric, F.Cu at (279.5, 225.4)
- added R8: R, Resistor_SMD:R_0805_2012Metric, F.Cu at (279.5, 118.1)
- added R9: R, Resistor_SMD:R_0805_2012Metric, F.Cu at (272.9, 209.0)
- added R9: R, Resistor_SMD:R_0805_2012Metric, F.Cu at (272.9, 101.7)
- added U1: EL817, Package_DIP:DIP-4_W7.62mm, F.Cu at (271.7, 170.1)
- added U1: EL817, Package_DIP:DIP-4_W7.62mm, F.Cu at (271.6, 62.8)
- added U2: EL817, Package_DIP:DIP-4_W7.62mm, F.Cu at (274.4, 150.7)
- added U2: EL817, Package_DIP:DIP-4_W7.62mm, F.Cu at (274.3, 43.4)
- added U3: EL817, Package_DIP:DIP-4_W7.62mm, F.Cu at (271.9, 200.7)
- added U3: EL817, Package_DIP:DIP-4_W7.62mm, F.Cu at (271.9, 93.3)
- added U4: EL817, Package_DIP:DIP-4_W7.62mm, F.Cu at (273.5, 111.9)
- added U4: EL817, Package_DIP:DIP-4_W7.62mm, F.Cu at (273.6, 219.2)
- added U5: L7805, MacroLib:TO-220-3_Vertical, F.Cu at (254.3, 47.7)
- added U5: L7805, MacroLib:TO-220-3_Vertical, F.Cu at (254.3, 155.0)
- added U6: ESP32DevKitv1, RF_Module:ESP32-C3-DevKitM-1, F.Cu at (237.5, 62.5)
- added U6: ESP32DevKitv1, RF_Module:ESP32-C3-DevKitM-1, F.Cu at (237.5, 169.8)
- moved C1 66.4 mm to (116.9, 47.2)
- moved C2 66.4 mm to (102.5, 47.2)
- moved D1 66.4 mm to (141.9, 49.7)
- moved D2 66.4 mm to (124.8, 49.7)
- moved D3 66.4 mm to (141.5, 92.3)
- moved D4 66.4 mm to (123.8, 100.3)
- moved D6 66.4 mm to (123.4, 68.7)
- moved D7 66.4 mm to (141.2, 112.5)
- moved D8 66.4 mm to (123.8, 119.4)
- moved J10 66.4 mm to (180.3, 64.2)
- moved J11 66.4 mm to (180.3, 73.9)
- moved J3 66.4 mm to (180.4, 45.4)
- moved J4 66.4 mm to (180.3, 113.0)
- moved J5 66.4 mm to (93.8, 40.7)
- moved J6 66.4 mm to (180.3, 92.0)
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Routing:
- net RV-VCC: track 355.8 -> 711.6 mm, vias 4 -> 12
- net GIOP36: track 69.6 -> 139.1 mm, vias 1 -> 3
- net GIOP35: track 57.9 -> 115.8 mm, vias 1 -> 3
- net GIOP39: track 55.0 -> 110.0 mm, vias 1 -> 3
- net GIOP34: track 52.2 -> 104.4 mm, vias 1 -> 3
- net Net-(D1-A): track 33.2 -> 67.9 mm, vias 1 -> 3
- net Net-(D3-A): track 39.3 -> 65.0 mm, vias 1 -> 3
- net Net-(D5-A): track 29.3 -> 53.1 mm, vias 1 -> 3
- net J8 - NC: track 23.8 -> 47.6 mm
- net Net-(D7-A): track 34.9 -> 58.7 mm, vias 1 -> 3
- net J4 - NC: track 23.5 -> 47.1 mm
- net J6 - NC: track 23.3 -> 46.7 mm
- net J2 - NC: track 21.8 -> 43.5 mm
- net J5 - NC: track 21.3 -> 42.5 mm
- net J3 - NC: track 21.1 -> 42.3 mm
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Other:
- board text added: "6°5° SIMÓN MIRANDA GASTÓN ARIEL EDUARDO PRIETO DIAZ"
