File: riliwifi-master/riliwifi-master/riliwifi-master/Hardware/relewifi-2025-05-13_163020/relewifi.kicad_sch (KiCad schematic)
At the start: 45 parts, among them J10 Screw_Terminal_01x03, J11 Screw_Terminal_01x03, J3 Screw_Terminal_01x03, J4 Screw_Terminal_01x03, J5 Screw_Terminal_01x02, J6 Screw_Terminal_01x03, J7 Screw_Terminal_01x03, J8 Screw_Terminal_01x03, J9 Screw_Terminal_01x03, K1 FINDER-40.52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

Commit message: Para imprimir
Parts:
- removed Q1, Q2, Q3, Q4: Q_NPN_BCE, Package_TO_SOT_SMD:SOT-416, symbol Device:Q_NPN_BCE
- added Q3, Q5, Q6, Q7: MMBT2222A, Package_TO_SOT_SMD:SOT-23, symbol Transistor_BJT:MMBT2222A
Connections:
- net GND: now also Q3.2 (E), Q5.2 (E), Q6.2 (E), Q7.2 (E)
- net at D3.2 (A), K3.A2, R9.1: now also Q6.3 (C)
- net at D7.2 (A), K4.A2, R12.1: now also Q5.3 (C)
- net at D1.2 (A), K1.A2, R10.1: now also Q7.3 (C)
- net at D5.2 (A), K2.A2, R11.1: now also Q3.3 (C)
- net at R8.2: now also Q5.1 (B)
- net at R2.2: now also Q6.1 (B)
- net at R4.2: now also Q3.1 (B)
- net at R7.2: now also Q7.1 (B)
